Commit message: 학습은 된다. 설계 문제

File: source/isaaclab_assets/isaaclab_assets/f1tenth/f1tenth.urdf (robot description, URDF)
Before this commit: robot f1tenth_racecar, 8 links, 7 joints
Joints:
- joint left_front_wheel_joint: limit (none) -> lower=-1e9 upper=1e9 effort=100.0 velocity=400.0; type continuous -> revolute
- joint left_rear_wheel_joint: limit (none) -> lower=-1e9 upper=1e9 effort=100.0 velocity=400.0; type continuous -> revolute
- joint right_front_wheel_joint: limit (none) -> lower=-1e9 upper=1e9 effort=100.0 velocity=400.0; type continuous -> revolute
- joint right_rear_wheel_joint: limit (none) -> lower=-1e9 upper=1e9 effort=100.0 velocity=400.0; type continuous -> revolute
